File: Ratibroombroom.sch (KiCad schematic (older format))
At the start: 113 parts, among them J1 Conn_01x02_Male, J10 Conn_01x04_Male, J11 Conn_01x04_Male, J2 Conn_01x02_Male, J3 Conn_01x04_Male, J4 Conn_01x04_Male, J5 Conn_01x02_Male, J6 Conn_01x02_Male, J7 Conn_01x04_Male, J8 Conn_01x04_Male, J9 Conn_01x04_Male, Q1 IRLML6344, Q10 S8050, Q11 IRF7416PbF, Q2 IRLML6344, Q3 IRLML6344, Q4 IRLML6344, Q5 PT12-21B/TR8, Q6 PT12-21B/TR8, Q7 PT12-21B/TR8, Q8 PT12-21B/TR8, Q9 IRLML6344, SW1 B3U, SW2 B3U, SW3 PCM12, U1 AZ1117-3.3, U2 DRV8835, U3 AS5145B-HSST, U4 MPU-9250, U5 STM32F405RGTx, U6 AS5145B-HSST, U7 DRV8835, U8 L6932D1.2TR, U9 L6932D1.2TR, Y1 8MHZ

Commit message: Added BOM parts for Power section
Parts:
- C1, C2, C21, C3, C4, C5, C6: MFR (none) -> 0603B105K100CT
- C10, C28, C29, C30, C31, C8: MFR (none) -> 0603X106K100NT
- J1: MFR (none) -> B2B-XH-A(LF)(SN)
- Q11: MFR (none) -> IRF7416TRPBF
- R1, R2: MFR (none) -> WR06X2612FTL
- R28, R30: MFR (none) -> RTT035601BTP
- R29, R31: MFR (none) -> 0603WAD1801T5E
- R3, R34: MFR (none) -> CR0603FA1002G
- SW3: MFR (none) -> PCM12SMTR
- U1: MFR (none) -> AZ1117H-3.3TRE1
- U8, U9: MFR (none) -> L6932D1.2TR
Changed lines of the file:
@@
 EESchema Schematic File Version 4
 LIBS:Ratibroombroom-cache
-EELAYER 29 0
+EELAYER 26 0
 EELAYER END
 $Descr A3 16535 11693
@@
 F 2 "Capacitor_SMD:C_0603_1608Metric" H 3538 1500 50  0001 C CNN
 F 3 "~" H 3500 1650 50  0001 C CNN
+F 4 "0603B105K100CT" H 3500 1650 50  0001 C CNN "MFR"
 	1    3500 1650
 	1    0    0    -1
@@
 F 2 "Capacitor_SMD:C_0603_1608Metric" H 4388 1500 50  0001 C CNN
 F 3 "~" H 4350 1650 50  0001 C CNN
+F 4 "0603B105K100CT" H 4350 1650 50  0001 C CNN "MFR"
 	1    4350 1650
 	1    0    0    -1
@@
 F 2 "Resistor_SMD:R_0603_1608Metric" V 3080 1500 50  0001 C CNN
 F 3 "~" H 3150 1500 50  0001 C CNN
+F 4 "CR0603FA1002G" H 3150 1500 50  0001 C CNN "MFR"
 	1    3150 1500
 	1    0    0    -1
@@
 F 2 "Connector_JST:JST_XH_B2B-XH-A_1x02_P2.50mm_Vertical" H 950 1300 50  0001 C CNN
 F 3 "~" H 950 1300 50  0001 C CNN
+F 4 "B2B-XH-A(LF)(SN)" H 950 1300 50  0001 C CNN "MFR"
 	1    950  1300
 	1    0    0    -1
@@
 F 2 "Resistor_SMD:R_0603_1608Metric" V 2330 1500 50  0001 C CNN
 F 3 "~" H 2400 1500 50  0001 C CNN
+F 4 "WR06X2612FTL" H 2400 1500 50  0001 C CNN "MFR"
 	1    2400 1500
 	1    0    0    -1
@@
 F 2 "Resistor_SMD:R_0603_1608Metric" V 2330 1800 50  0001 C CNN
 F 3 "~" H 2400 1800 50  0001 C CNN
+F 4 "WR06X2612FTL" H 2400 1800 50  0001 C CNN "MFR"
 	1    2400 1800
 	1    0    0    -1
@@
 F 2 "Package_TO_SOT_SMD:SOT-223-3_TabPin2" H 3950 1550 50  0001 C CIN
 F 3 "https://www.diodes.com/assets/Datasheets/AZ1117.pdf" H 3950 1300 50  0001 C CNN
+F 4 "AZ1117H-3.3TRE1" H 3950 1300 50  0001 C CNN "MFR"
 	1    3950 1300
 	1    0    0    -1
@@
 F 2 "Capacitor_SMD:C_0603_1608Metric" H 6688 1700 50  0001 C CNN
 F 3 "~" H 6650 1850 50  0001 C CNN
+F 4 "0603B105K100CT" H 6650 1850 50  0001 C CNN "MFR"
 	1    6650 1850
 	1    0    0    -1
@@
 F 2 "Capacitor_SMD:C_0603_1608Metric" H 8888 1700 50  0001 C CNN
 F 3 "~" H 8850 1850 50  0001 C CNN
+F 4 "0603B105K100CT" H 8850 1850 50  0001 C CNN "MFR"
 	1    8850 1850
 	1    0    0    -1
@@
 F 2 "Capacitor_SMD:C_0603_1608Metric" H 6688 3450 50  0001 C CNN
 F 3 "~" H 6650 3600 50  0001 C CNN
+F 4 "0603B105K100CT" H 6650 3600 50  0001 C CNN "MFR"
 	1    6650 3600
 	1    0    0    -1
@@
 F 2 "Capacitor_SMD:C_0603_1608Metric" H 8888 3450 50  0001 C CNN
 F 3 "~" H 8850 3600 50  0001 C CNN
+F 4 "0603B105K100CT" H 8850 3600 50  0001 C CNN "MFR"
 	1    8850 3600
 	1    0    0    -1
@@
 F 2 "Capacitor_SMD:C_0603_1608Metric" H 12588 1300 50  0001 C CNN
 F 3 "~" H 12550 1450 50  0001 C CNN
+F 4 "0603X106K100NT" H 12550 1450 50  0001 C CNN "MFR"
 	1    12550 1450
 	1    0    0    -1
@@
 F 2 "Capacitor_SMD:C_0603_1608Metric" H 4888 7050 50  0001 C CNN
 F 3 "~" H 4850 7200 50  0001 C CNN
+F 4 "0603B105K100CT" H 4850 7200 50  0001 C CNN "MFR"
 	1    4850 7200
 	-1   0    0    1
@@
 F 2 "Package_SO:SO-8_5.3x6.2mm_P1.27mm" H 2500 3125 50  0001 C CNN
 F 3 "https://www.st.com/resource/en/datasheet/l6932.pdf" H 2500 2800 50  0001 C CNN
+F 4 "L6932D1.2TR" H 2500 2800 50  0001 C CNN "MFR"
 	1    2500 2800
 	1    0    0    -1
@@
 F 2 "Resistor_SMD:R_0603_1608Metric" V 3030 2850 50  0001 C CNN
 F 3 "~" H 3100 2850 50  0001 C CNN
+F 4 "RTT035601BTP" H 3100 2850 50  0001 C CNN "MFR"
 	1    3100 2850
 	1    0    0    -1
@@
 F 2 "Resistor_SMD:R_0603_1608Metric" V 3030 3250 50  0001 C CNN
 F 3 "~" H 3100 3250 50  0001 C CNN
+F 4 "0603WAD1801T5E" H 3100 3250 50  0001 C CNN "MFR"
 	1    3100 3250
 	1    0    0    -1
@@
 F 2 "Capacitor_SMD:C_0603_1608Metric" H 3388 2900 50  0001 C CNN
 F 3 "~" H 3350 3050 50  0001 C CNN
+F 4 "0603X106K100NT" H 3350 3050 50  0001 C CNN "MFR"
 	1    3350 3050
 	-1   0    0    1
@@
 F 2 "Capacitor_SMD:C_0603_1608Metric" H 1988 2850 50  0001 C CNN
 F 3 "~" H 1950 3000 50  0001 C CNN
+F 4 "0603X106K100NT" H 1950 3000 50  0001 C CNN "MFR"
 	1    1950 3000
 	-1   0    0    1
@@
 F 2 "Package_SO:SO-8_5.3x6.2mm_P1.27mm" H 2500 4475 50  0001 C CNN
 F 3 "https://www.st.com/resource/en/datasheet/l6932.pdf" H 2500 4150 50  0001 C CNN
+F 4 "L6932D1.2TR" H 2500 4150 50  0001 C CNN "MFR"
 	1    2500 4150
 	1    0    0    -1
@@
 F 2 "Resistor_SMD:R_0603_1608Metric" V 3030 4200 50  0001 C CNN
 F 3 "~" H 3100 4200 50  0001 C CNN
+F 4 "RTT035601BTP" H 3100 4200 50  0001 C CNN "MFR"
 	1    3100 4200
 	1    0    0    -1
@@
 F 2 "Resistor_SMD:R_0603_1608Metric" V 3030 4600 50  0001 C CNN
 F 3 "~" H 3100 4600 50  0001 C CNN
+F 4 "0603WAD1801T5E" H 3100 4600 50  0001 C CNN "MFR"
 	1    3100 4600
 	1    0    0    -1
@@
 F 2 "Capacitor_SMD:C_0603_1608Metric" H 3388 4250 50  0001 C CNN
 F 3 "~" H 3350 4400 50  0001 C CNN
+F 4 "0603X106K100NT" H 3350 4400 50  0001 C CNN "MFR"
 	1    3350 4400
 	-1   0    0    1
@@
 F 2 "Capacitor_SMD:C_0603_1608Metric" H 1988 4200 50  0001 C CNN
 F 3 "~" H 1950 4350 50  0001 C CNN
+F 4 "0603X106K100NT" H 1950 4350 50  0001 C CNN "MFR"
 	1    1950 4350
 	-1   0    0    1
@@
 F 2 "Capacitor_SMD:C_0603_1608Metric" H 15238 1300 50  0001 C CNN
 F 3 "~" H 15200 1450 50  0001 C CNN
+F 4 "0603X106K100NT" H 15200 1450 50  0001 C CNN "MFR"
 	1    15200 1450
 	1    0    0    -1
@@
 F 2 "Package_SO:SO-8_5.3x6.2mm_P1.27mm" H 2150 1500 50  0001 C CNN
 F 3 "https://www.infineon.com/dgdl/irf7416pbf.pdf" H 1950 1400 50  0001 C CNN
+F 4 "IRF7416TRPBF" V 1950 1400 50  0001 C CNN "MFR"
 	1    1950 1400
 	0    1    -1   0
@@
 F 2 "Button_Switch_SMD:SW_SPDT_PCM12" H 1750 1850 50  0001 C CNN
 F 3 "~" H 1750 1850 50  0001 C CNN
+F 4 "PCM12SMTR" H 1750 1850 50  0001 C CNN "MFR"
 	1    1750 1850
 	-1   0    0    1
@@
 F 2 "Resistor_SMD:R_0603_1608Metric" V 1430 1500 50  0001 C CNN
 F 3 "~" H 1500 1500 50  0001 C CNN
+F 4 "CR0603FA1002G" H 1500 1500 50  0001 C CNN "MFR"
 	1    1500 1500
 	1    0    0    -1

Commit message: Added BOM parts for Motor control section
Parts:
- removed R20: 10k, Resistor_SMD:R_0603_1608Metric, symbol Device:R
- C12, C13, C19, C20, C22, C24, C25, C26, C7, C9: MFR (none) -> 0603B104K160CT
- Q9: MFR (none) -> IRLML6344TRPBF
- R21: MFR (none) -> WR06X1000FTL
- R22, R32, R33: MFR (none) -> CR0603FA1002G
Connections:
- wire segments 423 -> 420
Other:
- note added: "O DRV8835 non o atopo \nen TSSOP, estará ben a \nreferencia??"
- note added: "Os encoders non levan\ncondesador de desacoplo\nna súa PCB??"
- note removed: "Comentar cómo se vai\na integrar a PCB principal\ncoas dos encoders"
- note removed: "JP1 e JP2:\nse poden quedar\nabertos, valen \npara desconectar\nmotores"
- note removed: "R28, R29, R30, R31\nque sexan do 1% \nou mellor para que\nnon se desbalanceen\nas tensións dos motores"
Changed lines of the file:
@@
 F 2 "Capacitor_SMD:C_0603_1608Metric" H 11038 1300 50  0001 C CNN
 F 3 "~" H 11000 1450 50  0001 C CNN
+F 4 "0603B104K160CT" H 11000 1450 50  0001 C CNN "MFR"
 	1    11000 1450
 	1    0    0    -1
@@
 F 2 "Capacitor_SMD:C_0603_1608Metric" H 13088 6500 50  0001 C CNN
 F 3 "~" H 13050 6650 50  0001 C CNN
+F 4 "0603B104K160CT" H 13050 6650 50  0001 C CNN "MFR"
 	1    13050 6650
 	1    0    0    -1
@@
 F 2 "Capacitor_SMD:C_0603_1608Metric" H 12588 5150 50  0001 C CNN
 F 3 "~" H 12550 5300 50  0001 C CNN
+F 4 "0603B104K160CT" H 12550 5300 50  0001 C CNN "MFR"
 	1    12550 5300
 	1    0    0    -1
@@
 F 2 "Resistor_SMD:R_0603_1608Metric" V 12930 3700 50  0001 C CNN
 F 3 "~" H 13000 3700 50  0001 C CNN
+F 4 "WR06X1000FTL" H 13000 3700 50  0001 C CNN "MFR"
 	1    13000 3700
 	1    0    0    -1
@@
 F 2 "Resistor_SMD:R_0603_1608Metric" V 12930 4100 50  0001 C CNN
 F 3 "~" H 13000 4100 50  0001 C CNN
+F 4 "CR0603FA1002G" H 13000 4100 50  0001 C CNN "MFR"
 	1    13000 4100
 	1    0    0    -1
@@
 F 2 "Package_TO_SOT_SMD:SOT-23" H 13450 4000 50  0001 C CNN
 F 3 "~" H 13250 3900 50  0001 C CNN
+F 4 "IRLML6344TRPBF" H 13250 3900 50  0001 C CNN "MFR"
 	1    13250 3900
 	1    0    0    -1
@@
 F 3 "" H 13350 3250 50  0001 C CNN
 	1    13350 3250
-	1    0    0    -1
-$EndComp
-$Comp
-L Device:R R20
-U 1 1 5E53FDF5
-P 12650 3900
-F 0 "R20" H 12720 3946 50  0000 L CNN
-F 1 "10k" H 12720 3855 50  0000 L CNN
-F 2 "Resistor_SMD:R_0603_1608Metric" V 12580 3900 50  0001 C CNN
-F 3 "~" H 12650 3900 50  0001 C CNN
-	1    12650 3900
-	1    0    0    -1
-$EndComp
-$Comp
-L power:GND #PWR055
-U 1 1 5E5400FA
-P 12650 4300
-F 0 "#PWR055" H 12650 4050 50  0001 C CNN
-F 1 "GND" H 12655 4127 50  0000 C CNN
-F 2 "" H 12650 4300 50  0001 C CNN
-F 3 "" H 12650 4300 50  0001 C CNN
-	1    12650 4300
 	1    0    0    -1
 $EndComp
@@
 F 2 "Capacitor_SMD:C_0603_1608Metric" H 4538 8250 50  0001 C CNN
 F 3 "~" H 4500 8400 50  0001 C CNN
+F 4 "0603B104K160CT" H 4500 8400 50  0001 C CNN "MFR"
 	1    4500 8400
 	-1   0    0    1
@@
 F 2 "Capacitor_SMD:C_0603_1608Metric" H 4588 7050 50  0001 C CNN
 F 3 "~" H 4550 7200 50  0001 C CNN
+F 4 "0603B104K160CT" H 4550 7200 50  0001 C CNN "MFR"
 	1    4550 7200
 	-1   0    0    1
@@
 F 2 "Capacitor_SMD:C_0603_1608Metric" H 4888 8250 50  0001 C CNN
 F 3 "~" H 4850 8400 50  0001 C CNN
+F 4 "0603B104K160CT" H 4850 8400 50  0001 C CNN "MFR"
 	1    4850 8400
 	-1   0    0    1
@@
 F 2 "Capacitor_SMD:C_0603_1608Metric" H 5288 8250 50  0001 C CNN
 F 3 "~" H 5250 8400 50  0001 C CNN
+F 4 "0603B104K160CT" H 5250 8400 50  0001 C CNN "MFR"
 	1    5250 8400
 	-1   0    0    1
@@
 F 2 "Capacitor_SMD:C_0603_1608Metric" H 5688 8250 50  0001 C CNN
 F 3 "~" H 5650 8400 50  0001 C CNN
+F 4 "0603B104K160CT" H 5650 8400 50  0001 C CNN "MFR"
 	1    5650 8400
 	-1   0    0    1
@@
 F 2 "Capacitor_SMD:C_0603_1608Metric" H 5338 7050 50  0001 C CNN
 F 3 "~" H 5300 7200 50  0001 C CNN
+F 4 "0603B104K160CT" H 5300 7200 50  0001 C CNN "MFR"
 	1    5300 7200
 	-1   0    0    1
@@
 Wire Wire Line
 	13000 4250 13000 4300
-Wire Wire Line
-	12650 4050 12650 4300
 $Comp
 L Connector:Conn_01x04_Male J7
@@
 F 2 "Capacitor_SMD:C_0603_1608Metric" H 13688 1300 50  0001 C CNN
 F 3 "~" H 13650 1450 50  0001 C CNN
+F 4 "0603B104K160CT" H 13650 1450 50  0001 C CNN "MFR"
 	1    13650 1450
 	1    0    0    -1
@@
 Wire Notes Line
 	4750 4650 16000 4650
-Wire Wire Line
-	12650 3750 12650 3500
-Connection ~ 12650 3500
-Wire Wire Line
-	12650 3500 13000 3500
-Wire Wire Line
-	12100 3500 12650 3500
 $Comp
 L Device:R R33
@@
 F 2 "Resistor_SMD:R_0603_1608Metric" V 13805 2625 50  0001 C CNN
 F 3 "~" H 13875 2625 50  0001 C CNN
+F 4 "CR0603FA1002G" H 13875 2625 50  0001 C CNN "MFR"
 	1    13875 2625
 	1    0    0    -1
@@
 F 2 "Resistor_SMD:R_0603_1608Metric" V 11155 2600 50  0001 C CNN
 F 3 "~" H 11225 2600 50  0001 C CNN
+F 4 "CR0603FA1002G" H 11225 2600 50  0001 C CNN "MFR"
 	1    11225 2600
 	1    0    0    -1
@@
 Wire Wire Line
 	13875 2850 13875 2775
-Text Notes 3800 3650 0    50   ~ 0
-R28, R29, R30, R31\nque sexan do 1% \nou mellor para que\nnon se desbalanceen\nas tensións dos motores
-Text Notes 875  2975 0    50   ~ 0
-JP1 e JP2:\nse poden quedar\nabertos, valen \npara desconectar\nmotores
-Text Notes 10000 8275 0    50   ~ 0
-Comentar cómo se vai\na integrar a PCB principal\ncoas dos encoders
 Wire Wire Line
 	6650 1000 6200 1000
@@
 $EndComp
 Connection ~ 14450 8000
+Wire Wire Line
+	12100 3500 13000 3500
+Text Notes 12850 8200 0    50   ~ 0
+Os encoders non levan\ncondesador de desacoplo\nna súa PCB??
+Text Notes 12650 1875 0    50   ~ 0
+O DRV8835 non o atopo \nen TSSOP, estará ben a \nreferencia??
 $EndSCHEMATC
