File: Ratibroombroom.sch (KiCad schematic (older format))
At the start: 112 parts, among them J1 Conn_01x02_Male, J10 Conn_01x04_Male, J11 Conn_01x04_Male, J2 Conn_01x02_Male, J3 Conn_01x04_Male, J4 Conn_01x04_Male, J5 Conn_01x02_Male, J6 Conn_01x02_Male, J7 Conn_01x04_Male, J8 Conn_01x04_Male, J9 Conn_01x04_Male, Q1 IRLML6344, Q10 S8050, Q11 IRF7416PbF, Q2 IRLML6344, Q3 IRLML6344, Q4 IRLML6344, Q5 PT12-21B/TR8, Q6 PT12-21B/TR8, Q7 PT12-21B/TR8, Q8 PT12-21B/TR8, Q9 IRLML6344, SW1 B3U, SW2 B3U, SW3 PCM12, U1 AZ1117-3.3, U2 DRV8835, U3 AS5145B-HSST, U4 MPU-9250, U5 STM32F405RGTx, U6 AS5145B-HSST, U7 DRV8835, U8 L6932D1.2TR, U9 L6932D1.2TR, Y1 8MHZ

Commit message: Added BOM parts for IMU section
Parts:
- C11: MFR (none) -> C0603X7R103MDTS
- U4: MFR (none) -> MPU-9250
Changed lines of the file:
@@
 F 2 "Sensor_Motion:InvenSense_QFN-24_3x3mm_P0.4mm" H 11850 5200 50  0001 C CNN
 F 3 "https://store.invensense.com/datasheets/invensense/MPU9250REV1.0.pdf" H 11850 6050 50  0001 C CNN
+F 4 "MPU-9250" H 11850 6200 50  0001 C CNN "MFR"
 	1    11850 6200
 	1    0    0    -1
@@
 F 2 "Capacitor_SMD:C_0603_1608Metric" H 11088 5150 50  0001 C CNN
 F 3 "~" H 11050 5300 50  0001 C CNN
+F 4 "C0603X7R103MDTS" H 11050 5300 50  0001 C CNN "MFR"
 	1    11050 5300
 	1    0    0    -1

Commit message: Added BOM parts for Buzzer section
Parts:
- BZ1: MFR (none) -> MLT-5020
- D6: value 1N1418 -> 1N4148; MFR (none) -> 1N4148WS
- Q10: MFR (none) -> SS8050
- R24: MFR (none) -> CR0603FA1002G
Other:
- note added: "Cambio 1N1418 por 1N4148\nse me colei avisa"
Changed lines of the file:
@@
 F 2 "Package_TO_SOT_SMD:SOT-23" H 14900 6350 50  0001 C CNN
 F 3 "~" H 14700 6250 50  0001 C CNN
+F 4 "SS8050" H 14700 6250 50  0001 C CNN "MFR"
 	1    14700 6250
 	1    0    0    -1
@@
 F 2 "Ratibroombroom:MLT-5020" V 14975 5950 50  0001 C CNN
 F 3 "~" V 14975 5950 50  0001 C CNN
+F 4 "MLT-5020" H 15000 5850 50  0001 C CNN "MFR"
 	1    15000 5850
 	1    0    0    -1
@@
 P 14650 5850
 F 0 "D6" V 14500 5500 50  0000 L CNN
-F 1 "1N1418" V 14600 5500 50  0000 L CNN
+F 1 "1N4148" V 14600 5500 50  0000 L CNN
 F 2 "Diode_SMD:D_SOD-323" H 14650 5850 50  0001 C CNN
 F 3 "~" H 14650 5850 50  0001 C CNN
+F 4 "1N4148WS" V 14650 5850 50  0001 C CNN "MFR"
 	1    14650 5850
 	0    1    1    0
@@
 F 2 "Resistor_SMD:R_0603_1608Metric" V 14230 6250 50  0001 C CNN
 F 3 "~" H 14300 6250 50  0001 C CNN
+F 4 "CR0603FA1002G" V 14300 6250 50  0001 C CNN "MFR"
 	1    14300 6250
 	0    1    1    0
@@
 Text Notes 12650 1875 0    50   ~ 0
 O DRV8835 non o atopo \nen TSSOP, estará ben a \nreferencia??
+Text Notes 13600 5650 0    50   ~ 0
+Cambio 1N1418 por 1N4148\nse me colei avisa
 $EndSCHEMATC

Commit message: Added BOM parts for Button and LED sections
Parts:
- C16, C27: MFR (none) -> C0603X7R103MDTS
- R23, R25, R26, R27: MFR (none) -> WR06X1000FTL
- SW1, SW2: MFR (none) -> B3U-1000P
Other:
- note added: "Decidir color LEDs"
Changed lines of the file:
@@
 F 2 "Resistor_SMD:R_0603_1608Metric" V 8830 9750 50  0001 C CNN
 F 3 "~" H 8900 9750 50  0001 C CNN
+F 4 "WR06X1000FTL" H 8900 9750 50  0001 C CNN "MFR"
 	1    8900 9750
 	1    0    0    -1
@@
 F 2 "Resistor_SMD:R_0603_1608Metric" V 9180 9750 50  0001 C CNN
 F 3 "~" H 9250 9750 50  0001 C CNN
+F 4 "WR06X1000FTL" H 9250 9750 50  0001 C CNN "MFR"
 	1    9250 9750
 	1    0    0    -1
@@
 F 2 "Resistor_SMD:R_0603_1608Metric" V 9530 9750 50  0001 C CNN
 F 3 "~" H 9600 9750 50  0001 C CNN
+F 4 "WR06X1000FTL" H 9600 9750 50  0001 C CNN "MFR"
 	1    9600 9750
 	1    0    0    -1
@@
 F 2 "Resistor_SMD:R_0603_1608Metric" V 9880 9750 50  0001 C CNN
 F 3 "~" H 9950 9750 50  0001 C CNN
+F 4 "WR06X1000FTL" H 9950 9750 50  0001 C CNN "MFR"
 	1    9950 9750
 	1    0    0    -1
@@
 F 2 "Button_Switch_SMD:SW_SPST_B3U-1000P" H 6900 10150 50  0001 C CNN
 F 3 "~" H 6900 10150 50  0001 C CNN
+F 4 "B3U-1000P" V 6900 9950 50  0001 C CNN "MFR"
 	1    6900 9950
 	0    1    1    0
@@
 F 2 "Capacitor_SMD:C_0603_1608Metric" H 6588 9800 50  0001 C CNN
 F 3 "~" H 6550 9950 50  0001 C CNN
+F 4 "C0603X7R103MDTS" H 6550 9950 50  0001 C CNN "MFR"
 	1    6550 9950
 	1    0    0    -1
@@
 F 2 "Button_Switch_SMD:SW_SPST_B3U-1000P" H 7850 10150 50  0001 C CNN
 F 3 "~" H 7850 10150 50  0001 C CNN
+F 4 "B3U-1000P" V 7850 9950 50  0001 C CNN "MFR"
 	1    7850 9950
 	0    1    1    0
@@
 F 2 "Capacitor_SMD:C_0603_1608Metric" H 7538 9800 50  0001 C CNN
 F 3 "~" H 7500 9950 50  0001 C CNN
+F 4 "C0603X7R103MDTS" H 7500 9950 50  0001 C CNN "MFR"
 	1    7500 9950
 	1    0    0    -1
@@
 Text Notes 13600 5650 0    50   ~ 0
 Cambio 1N1418 por 1N4148\nse me colei avisa
+Text Notes 9125 10700 0    50   ~ 0
+Decidir color LEDs
 $EndSCHEMATC

Commit message: Added BOM parts for Microcontroller section
Parts:
- C14, C15: MFR (none) -> CL10C200JB8NNNC
- C17, C18: MFR (none) -> CL10B225KP8NNNC
- C23: MFR (none) -> 0603B475K100NT
- U5: MFR (none) -> STM32F405RGT6
- Y1: MFR (none) -> XVGCELNANF-8.000
Other:
- note added: "Revisar referencia\ncristal"
Changed lines of the file:
@@
 F 2 "Package_QFP:LQFP-64_10x10mm_P0.5mm" H 2100 6850 50  0001 R CNN
 F 3 "http://www.st.com/st-web-ui/static/active/en/resource/technical/document/datasheet/DM00037051.pdf" H 2700 8550 50  0001 C CNN
+F 4 "STM32F405RGT6" H 2700 8550 50  0001 C CNN "MFR"
 	1    2700 8550
 	1    0    0    -1
@@
 F 2 "Crystal:Crystal_SMD_5032-4Pin_5.0x3.2mm" H 5000 9500 50  0001 C CNN
 F 3 "~" H 5000 9500 50  0001 C CNN
+F 4 "XVGCELNANF-8.000" V 5000 9500 50  0001 C CNN "MFR"
 	1    5000 9500
 	0    1    1    0
@@
 F 2 "Capacitor_SMD:C_0603_1608Metric" H 4738 9600 50  0001 C CNN
 F 3 "~" H 4700 9750 50  0001 C CNN
+F 4 "CL10C200JB8NNNC" V 4700 9750 50  0001 C CNN "MFR"
 	1    4700 9750
 	0    1    1    0
@@
 F 2 "Capacitor_SMD:C_0603_1608Metric" H 4738 9100 50  0001 C CNN
 F 3 "~" H 4700 9250 50  0001 C CNN
+F 4 "CL10C200JB8NNNC" V 4700 9250 50  0001 C CNN "MFR"
 	1    4700 9250
 	0    1    1    0
@@
 F 2 "Capacitor_SMD:C_0603_1608Metric" H 1488 7350 50  0001 C CNN
 F 3 "~" H 1450 7500 50  0001 C CNN
+F 4 "CL10B225KP8NNNC" H 1450 7500 50  0001 C CNN "MFR"
 	1    1450 7500
 	-1   0    0    1
@@
 F 2 "Capacitor_SMD:C_0603_1608Metric" H 5638 7050 50  0001 C CNN
 F 3 "~" H 5600 7200 50  0001 C CNN
+F 4 "0603B475K100NT" H 5600 7200 50  0001 C CNN "MFR"
 	1    5600 7200
 	-1   0    0    1
@@
 F 2 "Capacitor_SMD:C_0603_1608Metric" H 1738 7450 50  0001 C CNN
 F 3 "~" H 1700 7600 50  0001 C CNN
+F 4 "CL10B225KP8NNNC" H 1700 7600 50  0001 C CNN "MFR"
 	1    1700 7600
 	-1   0    0    1
@@
 Text Notes 9125 10700 0    50   ~ 0
 Decidir color LEDs
+Text Notes 5450 9500 0    50   ~ 0
+Revisar referencia\ncristal
 $EndSCHEMATC

Commit message: Added BOM parts for Encoder section
Parts:
- U3, U6: MFR (none) -> AS5145B-HSSM
Changed lines of the file:
@@
 F 2 "Package_SO:SSOP-16_5.3x6.2mm_P0.65mm" H 12150 9200 50  0001 C CNN
 F 3 "https://ams.com/documents/20143/36005/AS5145_DS000398_1-00.pdf" H 12150 9200 50  0001 C CNN
+F 4 "AS5145B-HSSM" H 12150 8750 50  0001 C CNN "MFR"
 	1    12150 8750
 	1    0    0    -1
@@
 F 2 "Package_SO:SSOP-16_5.3x6.2mm_P0.65mm" H 14400 9200 50  0001 C CNN
 F 3 "https://ams.com/documents/20143/36005/AS5145_DS000398_1-00.pdf" H 14400 9200 50  0001 C CNN
+F 4 "AS5145B-HSSM" H 14400 8750 50  0001 C CNN "MFR"
 	1    14400 8750
 	1    0    0    -1

Commit message: Added BOM parts for Wall Sensor section
Parts:
- Q1, Q2, Q3, Q4: MFR (none) -> IRLML6344TRPBF
- Q5, Q6, Q7, Q8: MFR (none) -> PT12-21B/TR8
- R12, R16, R4, R8: MFR (none) -> WR06X1000FTL
- R13, R17, R5, R9: MFR (none) -> CR0603FA1003G
Changed lines of the file:
@@
 F 2 "Ratibroombroom:PT12-21B-TR8" H 7250 1750 50  0001 C CNN
 F 3 "~" H 7050 1650 50  0001 C CNN
+F 4 "PT12-21B/TR8" H 7050 1650 50  0001 C CNN "MFR"
 	1    7050 1650
 	1    0    0    -1
@@
 F 2 "Resistor_SMD:R_0603_1608Metric" V 5780 1650 50  0001 C CNN
 F 3 "~" H 5850 1650 50  0001 C CNN
+F 4 "WR06X1000FTL" H 5850 1650 50  0001 C CNN "MFR"
 	1    5850 1650
 	1    0    0    -1
@@
 F 2 "Resistor_SMD:R_0603_1608Metric" V 5780 2050 50  0001 C CNN
 F 3 "~" H 5850 2050 50  0001 C CNN
+F 4 "CR0603FA1003G" H 5850 2050 50  0001 C CNN "MFR"
 	1    5850 2050
 	1    0    0    -1
@@
 F 2 "Package_TO_SOT_SMD:SOT-23" H 6300 1950 50  0001 C CNN
 F 3 "~" H 6100 1850 50  0001 C CNN
+F 4 "IRLML6344TRPBF" H 6100 1850 50  0001 C CNN "MFR"
 	1    6100 1850
 	1    0    0    -1
@@
 F 2 "Ratibroombroom:PT12-21B-TR8" H 9450 1750 50  0001 C CNN
 F 3 "~" H 9250 1650 50  0001 C CNN
+F 4 "PT12-21B/TR8" H 9250 1650 50  0001 C CNN "MFR"
 	1    9250 1650
 	1    0    0    -1
@@
 F 2 "Resistor_SMD:R_0603_1608Metric" V 7980 1650 50  0001 C CNN
 F 3 "~" H 8050 1650 50  0001 C CNN
+F 4 "WR06X1000FTL" H 8050 1650 50  0001 C CNN "MFR"
 	1    8050 1650
 	1    0    0    -1
@@
 F 2 "Resistor_SMD:R_0603_1608Metric" V 7980 2050 50  0001 C CNN
 F 3 "~" H 8050 2050 50  0001 C CNN
+F 4 "CR0603FA1003G" H 8050 2050 50  0001 C CNN "MFR"
 	1    8050 2050
 	1    0    0    -1
@@
 F 2 "Package_TO_SOT_SMD:SOT-23" H 8500 1950 50  0001 C CNN
 F 3 "~" H 8300 1850 50  0001 C CNN
+F 4 "IRLML6344TRPBF" H 8300 1850 50  0001 C CNN "MFR"
 	1    8300 1850
 	1    0    0    -1
@@
 F 2 "Ratibroombroom:PT12-21B-TR8" H 7250 3500 50  0001 C CNN
 F 3 "~" H 7050 3400 50  0001 C CNN
+F 4 "PT12-21B/TR8" H 7050 3400 50  0001 C CNN "MFR"
 	1    7050 3400
 	1    0    0    -1
@@
 F 2 "Resistor_SMD:R_0603_1608Metric" V 5780 3400 50  0001 C CNN
 F 3 "~" H 5850 3400 50  0001 C CNN
+F 4 "WR06X1000FTL" H 5850 3400 50  0001 C CNN "MFR"
 	1    5850 3400
 	1    0    0    -1
@@
 F 2 "Resistor_SMD:R_0603_1608Metric" V 5780 3800 50  0001 C CNN
 F 3 "~" H 5850 3800 50  0001 C CNN
+F 4 "CR0603FA1003G" H 5850 3800 50  0001 C CNN "MFR"
 	1    5850 3800
 	1    0    0    -1
@@
 F 2 "Package_TO_SOT_SMD:SOT-23" H 6300 3700 50  0001 C CNN
 F 3 "~" H 6100 3600 50  0001 C CNN
+F 4 "IRLML6344TRPBF" H 6100 3600 50  0001 C CNN "MFR"
 	1    6100 3600
 	1    0    0    -1
@@
 F 2 "Ratibroombroom:PT12-21B-TR8" H 9450 3500 50  0001 C CNN
 F 3 "~" H 9250 3400 50  0001 C CNN
+F 4 "PT12-21B/TR8" H 9250 3400 50  0001 C CNN "MFR"
 	1    9250 3400
 	1    0    0    -1
@@
 F 2 "Resistor_SMD:R_0603_1608Metric" V 7980 3400 50  0001 C CNN
 F 3 "~" H 8050 3400 50  0001 C CNN
+F 4 "WR06X1000FTL" H 8050 3400 50  0001 C CNN "MFR"
 	1    8050 3400
 	1    0    0    -1
@@
 F 2 "Resistor_SMD:R_0603_1608Metric" V 7980 3800 50  0001 C CNN
 F 3 "~" H 8050 3800 50  0001 C CNN
+F 4 "CR0603FA1003G" H 8050 3800 50  0001 C CNN "MFR"
 	1    8050 3800
 	1    0    0    -1
@@
 F 2 "Package_TO_SOT_SMD:SOT-23" H 8500 3700 50  0001 C CNN
 F 3 "~" H 8300 3600 50  0001 C CNN
+F 4 "IRLML6344TRPBF" H 8300 3600 50  0001 C CNN "MFR"
 	1    8300 3600
 	1    0    0    -1

Commit message: Added BOM parts for Wall sensor section
Parts:
- D2, D3, D4, D5: MFR (none) -> SFH4045N
Changed lines of the file:
@@
 F 2 "Ratibroombroom:SFH4045N" H 6200 1450 50  0001 C CNN
 F 3 "~" H 6200 1450 50  0001 C CNN
+F 4 "SFH4045N" V 6200 1450 50  0001 C CNN "MFR"
 	1    6200 1450
 	0    -1   -1   0
@@
 F 2 "Ratibroombroom:SFH4045N" H 8400 1450 50  0001 C CNN
 F 3 "~" H 8400 1450 50  0001 C CNN
+F 4 "SFH4045N" V 8400 1450 50  0001 C CNN "MFR"
 	1    8400 1450
 	0    -1   -1   0
@@
 F 2 "Ratibroombroom:SFH4045N" H 6200 3200 50  0001 C CNN
 F 3 "~" H 6200 3200 50  0001 C CNN
+F 4 "SFH4045N" V 6200 3200 50  0001 C CNN "MFR"
 	1    6200 3200
 	0    -1   -1   0
@@
 F 2 "Ratibroombroom:SFH4045N" H 8400 3200 50  0001 C CNN
 F 3 "~" H 8400 3200 50  0001 C CNN
+F 4 "SFH4045N" V 8400 3200 50  0001 C CNN "MFR"
 	1    8400 3200
 	0    -1   -1   0

Commit message: Fix wrong footpring for DRV8835
Parts:
- U7: footprint Package_SO:TSSOP-16_4.4x5mm_P0.65mm -> Package_SON:WSON-12-1EP_3x2mm_P0.5mm_EP1x2.65_ThermalVias; MFR (none) -> DRV8835DSSR
Other:
- note removed: "O DRV8835 non o atopo \nen TSSOP, estará ben a \nreferencia??"
Changed lines of the file:
@@
 EESchema Schematic File Version 4
 LIBS:Ratibroombroom-cache
-EELAYER 26 0
+EELAYER 29 0
 EELAYER END
 $Descr A3 16535 11693
@@
 F 1 "DRV8835" H 11650 1450 50  0000 C CNN
 F 2 "Package_SO:TSSOP-16_4.4x5mm_P0.65mm" H 12350 2600 50  0001 L CNN
-F 3 "" H 11750 2700 50  0001 C CNN
+F 3 "DRV8835DSSR" H 11750 2700 50  0001 C CNN
 	1    11900 2150
 	1    0    0    -1
@@
 F 0 "U7" H 14200 1550 50  0000 C CNN
 F 1 "DRV8835" H 14300 1450 50  0000 C CNN
-F 2 "Package_SO:TSSOP-16_4.4x5mm_P0.65mm" H 15000 2600 50  0001 L CNN
+F 2 "Package_SON:WSON-12-1EP_3x2mm_P0.5mm_EP1x2.65_ThermalVias" H 15000 2600 50  0001 L CNN
 F 3 "" H 14400 2700 50  0001 C CNN
+F 4 "DRV8835DSSR" H 14550 2150 50  0001 C CNN "MFR"
 	1    14550 2150
 	1    0    0    -1
@@
 Text Notes 12850 8200 0    50   ~ 0
 Os encoders non levan\ncondesador de desacoplo\nna súa PCB??
-Text Notes 12650 1875 0    50   ~ 0
-O DRV8835 non o atopo \nen TSSOP, estará ben a \nreferencia??
 Text Notes 13600 5650 0    50   ~ 0
 Cambio 1N1418 por 1N4148\nse me colei avisa
